Commit message: Auto commit and push

File: install/canopen_tests/share/canopen_tests/urdf/canopen_system/canopen_system.ros2_control.xacro (robot description, xacro)
@@ -1,26 +1 @@
-<?xml version="1.0"?>
-<robot xmlns:xacro="http://www.ros.org/wiki/xacro">
-    <xacro:macro name="canopen_ros2_control_test" params="
-      name
-      prefix
-      bus_config
-      master_config
-      can_interface_name
-      master_bin">
-        <ros2_control name="${name}" type="system">
-            <hardware>
-              <plugin>canopen_ros2_control/CanopenSystem</plugin>
-              <param name="bus_config">${bus_config}</param>
-              <param name="master_config">${master_config}</param>
-              <param name="can_interface_name">${can_interface_name}</param>
-              <param name="master_bin">"${master_bin}"</param>
-            </hardware>
-            <joint name="${prefix}node_1">
-                <param name="node_id">2</param>
-            </joint>
-            <joint name="${prefix}node_2">
-                <param name="node_id">3</param>
-            </joint>
-        </ros2_control>
-    </xacro:macro>
-</robot>
+/home/ub2004/ros2_ws/src/ros2_canopen/canopen_tests/urdf/canopen_system/canopen_system.ros2_control.xacro

File: install/canopen_tests/share/canopen_tests/urdf/canopen_system/canopen_system.urdf.xacro (robot description, xacro)
@@ -1,41 +1 @@
-<?xml version="1.0"?>
-<robot xmlns:xacro="http://www.ros.org/wiki/xacro" name="$(arg name)">
-    <xacro:arg name="name" default="canopen_test_system"/>
-    <xacro:arg name="prefix" default="" />
-    <xacro:arg name="bus_config" default="$(find canopen_proxy_driver)/config/pdo_test/pdo.yml"/>
-    <xacro:arg name="master_config" default="$(find canopen_proxy_driver)/config/pdo_test/master.dcf"/>
-    <xacro:arg name="can_interface_name" default="vcan0"/>
-    <xacro:arg name="master_bin" default=""/>
-    <!-- ros2 control include -->
-    <xacro:include filename="$(find canopen_tests)/urdf/canopen_system/canopen_system.ros2_control.xacro"/>
-    <xacro:canopen_ros2_control_test
-      name="$(arg name)"
-      prefix="$(arg prefix)"
-      bus_config="$(arg bus_config)"
-      master_config="$(arg master_config)"
-      can_interface_name="$(arg can_interface_name)"
-      master_bin="$(arg master_bin)"
-    />
-    <link name="$(arg prefix)base_link"/>
-    <link name="$(arg prefix)node_1_link">
-      <visual>
-        <origin xyz="0 0 0" rpy="0 0 0"/>
-        <geometry>
-          <cylinder radius="0.1" length="1.0"/>
-        </geometry>
-      </visual>
-      <collision>
-        <origin xyz="0 0 0" rpy="0 0 0"/>
-        <geometry>
-          <cylinder radius="0.1" length="1.0"/>
-        </geometry>
-      </collision>
-    </link>
-    <joint name="$(arg prefix)node_1" type="revolute">
-        <parent link="$(arg prefix)base_link" />
-        <child link="$(arg prefix)node_1_link" />
-        <origin xyz="0 0 0" rpy="0 0 0" />
-        <axis xyz="0 0 1" />
-        <limit lower="${-2*pi}" upper="${2*pi}" effort="10.0" velocity="0.5"/>
-    </joint>
-</robot>
+/home/ub2004/ros2_ws/src/ros2_canopen/canopen_tests/urdf/canopen_system/canopen_system.urdf.xacro

File: install/canopen_tests/share/canopen_tests/urdf/cia402_system/cia402_system.ros2_control.xacro (robot description, xacro)
@@ -1,26 +1 @@
-<?xml version="1.0"?>
-<robot xmlns:xacro="http://www.ros.org/wiki/xacro">
-    <xacro:macro name="cia402_ros2_control_test" params="
-      name
-      prefix
-      bus_config
-      master_config
-      can_interface_name
-      master_bin">
-        <ros2_control name="${name}" type="system">
-            <hardware>
-              <plugin>canopen_ros2_control/Cia402System</plugin>
-              <param name="bus_config">${bus_config}</param>
-              <param name="master_config">${master_config}</param>
-              <param name="can_interface_name">${can_interface_name}</param>
-              <param name="master_bin">"${master_bin}"</param>
-            </hardware>
-            <joint name="${prefix}node_1">
-                <param name="node_id">2</param>
-            </joint>
-<!--            <joint name="${prefix}node_2">-->
-<!--                <param name="node_id">3</param>-->
-<!--            </joint>-->
-        </ros2_control>
-    </xacro:macro>
-</robot>
+/home/ub2004/ros2_ws/src/ros2_canopen/canopen_tests/urdf/cia402_system/cia402_system.ros2_control.xacro

File: install/canopen_tests/share/canopen_tests/urdf/cia402_system/cia402_system.urdf.xacro (robot description, xacro)
@@ -1,41 +1 @@
-<?xml version="1.0"?>
-<robot xmlns:xacro="http://www.ros.org/wiki/xacro" name="$(arg name)">
-    <xacro:arg name="name" default="cia402_test_system"/>
-    <xacro:arg name="prefix" default="" />
-    <xacro:arg name="bus_config" default="$(find canopen_tests)/config/cia402/bus.yml"/>
-    <xacro:arg name="master_config" default="$(find canopen_tests)/config/cia402/master.dcf"/>
-    <xacro:arg name="can_interface_name" default="vcan0"/>
-    <xacro:arg name="master_bin" default=""/>
-    <!-- ros2 control include -->
-    <xacro:include filename="$(find canopen_tests)/urdf/cia402_system/cia402_system.ros2_control.xacro"/>
-    <xacro:cia402_ros2_control_test
-      name="$(arg name)"
-      prefix="$(arg prefix)"
-      bus_config="$(arg bus_config)"
-      master_config="$(arg master_config)"
-      can_interface_name="$(arg can_interface_name)"
-      master_bin="$(arg master_bin)"
-    />
-    <link name="$(arg prefix)base_link"/>
-    <link name="$(arg prefix)node_1_link">
-      <visual>
-        <origin xyz="0 0 0" rpy="0 0 0"/>
-        <geometry>
-          <cylinder radius="0.1" length="1.0"/>
-        </geometry>
-      </visual>
-      <collision>
-        <origin xyz="0 0 0" rpy="0 0 0"/>
-        <geometry>
-          <cylinder radius="0.1" length="1.0"/>
-        </geometry>
-      </collision>
-    </link>
-    <joint name="$(arg prefix)node_1" type="revolute">
-        <parent link="$(arg prefix)base_link" />
-        <child link="$(arg prefix)node_1_link" />
-        <origin xyz="0 0 0" rpy="0 0 0" />
-        <axis xyz="0 0 1" />
-        <limit lower="${-2*pi}" upper="${2*pi}" effort="10.0" velocity="0.5"/>
-    </joint>
-</robot>
+/home/ub2004/ros2_ws/src/ros2_canopen/canopen_tests/urdf/cia402_system/cia402_system.urdf.xacro

File: install/canopen_tests/share/canopen_tests/urdf/robot_controller/robot_controller.macro.xacro (robot description, xacro)
@@ -1,67 +1 @@
-<?xml version="1.0"?>
-<robot xmlns:xacro="http://www.ros.org/wiki/xacro">
-    <xacro:macro name="robot_control_robot" params="
-        name
-        prefix
-        parent
-        *origin
-        " >
-    <link name="${prefix}link1">
-        <visual>
-            <origin xyz="0 0 0" rpy="0 0 0"/>
-            <geometry>
-                <cylinder radius="0.2" length="0.5"/>
-            </geometry>
-        </visual>
-    </link>
-    <link name="${prefix}link2">
-        <visual>
-            <origin xyz="0 0 0" rpy="0 0 0"/>
-            <geometry>
-                <cylinder radius="0.2" length="0.5"/>
-            </geometry>
-        </visual>
-    </link>
-    <link name="${prefix}link3">
-        <visual>
-            <origin xyz="0 0 0" rpy="0 0 0"/>
-            <geometry>
-                <cylinder radius="0.2" length="0.5"/>
-            </geometry>
-        </visual>
-    </link>
-    <link name="${prefix}link4">
-        <visual>
-            <origin xyz="0 0 0" rpy="0 0 0"/>
-            <geometry>
-                <cylinder radius="0.2" length="0.5"/>
-            </geometry>
-        </visual>
-    </link>
-    <joint name="${prefix}base_joint" type="fixed">
-        <xacro:insert_block name="origin" />
-        <parent link="${parent}"/>
-        <child link="${prefix}link1"/>
-    </joint>
-    <joint name="${prefix}joint1" type="revolute">
-        <parent link="${prefix}link1"/>
-        <child link="${prefix}link2"/>
-        <origin xyz="0 0 0.5" rpy="0 0 0"/>
-        <axis xyz="0 1 0" />
-        <limit lower="${-2*pi}" upper="${2*pi}" effort="10.0" velocity="0.5"/>
-    </joint>
-    <joint name="${prefix}joint2" type="revolute">
-        <parent link="${prefix}link2"/>
-        <child link="${prefix}link3"/>
-        <origin xyz="0 0 0.5" rpy="0 0 0"/>
-        <axis xyz="0 1 0" />
-        <limit lower="${-2*pi}" upper="${2*pi}" effort="10.0" velocity="0.5"/>
-    </joint>
-    <joint name="${prefix}joint3" type="fixed">
-        <parent link="${prefix}link3"/>
-        <child link="${prefix}link4"/>
-        <origin xyz="0 0 0.5" rpy="0 0 0"/>
-        <axis xyz="0 1 0" />
-    </joint>
-    </xacro:macro>
-</robot>
+/home/ub2004/ros2_ws/src/ros2_canopen/canopen_tests/urdf/robot_controller/robot_controller.macro.xacro

File: install/canopen_tests/share/canopen_tests/urdf/robot_controller/robot_controller.ros2_control.xacro (robot description, xacro)
@@ -1,28 +1 @@
-<?xml version="1.0"?>
-<robot xmlns:xacro="http://www.ros.org/wiki/xacro">
-    <xacro:macro name="robot_control_control" params="
-      name
-      prefix
-      bus_config
-      master_config
-      can_interface_name
-      master_bin">
-        <ros2_control name="${name}" type="system">
-            <hardware>
-              <plugin>canopen_ros2_control/RobotSystem</plugin>
-              <param name="bus_config">${bus_config}</param>
-              <param name="master_config">${master_config}</param>
-              <param name="can_interface_name">${can_interface_name}</param>
-              <param name="master_bin">"${master_bin}"</param>
-            </hardware>
-            <joint name="${prefix}joint1">
-                <param name="device_name">joint_1</param>
-                <state_interface name="position" />
-            </joint>
-            <joint name="${prefix}joint2">
-                <param name="device_name">joint_2</param>
-                <state_interface name="position" />
-            </joint>
-        </ros2_control>
-    </xacro:macro>
-</robot>
+/home/ub2004/ros2_ws/src/ros2_canopen/canopen_tests/urdf/robot_controller/robot_controller.ros2_control.xacro

File: install/canopen_tests/share/canopen_tests/urdf/robot_controller/robot_controller.urdf.xacro (robot description, xacro)
@@ -1,20 +1 @@
-<?xml version="1.0"?>
-<robot xmlns:xacro="http://wiki.ros.org/xacro" name="test_robot">
-    <xacro:include filename="$(find canopen_tests)/urdf/robot_controller/robot_controller.macro.xacro"/>
-    <xacro:include filename="$(find canopen_tests)/urdf/robot_controller/robot_controller.ros2_control.xacro"/>
-    <link name="world" />
-    <xacro:robot_control_robot
-        name="test_robot"
-        prefix=""
-        parent="world"
-        >
-            <origin xyz="0 0 0" rpy="0 0 0" />
-    </xacro:robot_control_robot>
-    <xacro:robot_control_control
-        name="test_robot"
-        prefix=""
-        bus_config="$(find canopen_tests)/config/robot_control/bus.yml"
-        master_config="$(find canopen_tests)/config/robot_control/master.dcf"
-        can_interface_name="vcan0"
-        master_bin="" />
-</robot>
+/home/ub2004/ros2_ws/src/ros2_canopen/canopen_tests/urdf/robot_controller/robot_controller.urdf.xacro

File: install/urdf_tutorial/share/urdf_tutorial/urdf/robot.xacro (robot description, xacro)
@@ -1,169 +1 @@
-<?xml version="1.0"?>
-<robot name="visual">
-  <material name="blue">
-    <color rgba="0 0 0.8 1"/>
-  </material>
-  <material name="black">
-    <color rgba="0 0 0 1"/>
-  </material>
-  <material name="white">
-    <color rgba="1 1 1 1"/>
-  </material>
-  <link name="base_link">
-    <visual>
-      <geometry>
-        <cylinder length="0.6" radius="0.2"/>
-      </geometry>
-      <material name="blue"/>
-    </visual>
-  </link>
-  <link name="right_leg">
-    <visual>
-      <geometry>
-        <box size="0.6 0.1 0.2"/>
-      </geometry>
-      <origin rpy="0 1.57075 0" xyz="0 0 -0.3"/>
-      <material name="white"/>
-    </visual>
-  </link>
-  <joint name="base_to_right_leg" type="fixed">
-    <parent link="base_link"/>
-    <child link="right_leg"/>
-    <origin xyz="0 -0.22 0.25"/>
-  </joint>
-  <link name="right_base">
-    <visual>
-      <geometry>
-        <box size="0.4 0.1 0.1"/>
-      </geometry>
-      <material name="white"/>
-    </visual>
-  </link>
-  <joint name="right_base_joint" type="fixed">
-    <parent link="right_leg"/>
-    <child link="right_base"/>
-    <origin xyz="0 0 -0.6"/>
-  </joint>
-  <link name="right_front_wheel">
-    <visual>
-      <origin rpy="1.57075 0 0" xyz="0 0 0"/>
-      <geometry>
-        <cylinder length="0.1" radius="0.035"/>
-      </geometry>
-      <material name="black"/>
-    </visual>
-  </link>
-  <joint name="right_front_wheel_joint" type="fixed">
-    <parent link="right_base"/>
-    <child link="right_front_wheel"/>
-    <origin rpy="0 0 0" xyz="0.133333333333 0 -0.085"/>
-  </joint>
-  <link name="right_back_wheel">
-    <visual>
-      <origin rpy="1.57075 0 0" xyz="0 0 0"/>
-      <geometry>
-        <cylinder length="0.1" radius="0.035"/>
-      </geometry>
-      <material name="black"/>
-    </visual>
-  </link>
-  <joint name="right_back_wheel_joint" type="fixed">
-    <parent link="right_base"/>
-    <child link="right_back_wheel"/>
-    <origin rpy="0 0 0" xyz="-0.133333333333 0 -0.085"/>
-  </joint>
-  <link name="left_leg">
-    <visual>
-      <geometry>
-        <box size="0.6 0.1 0.2"/>
-      </geometry>
-      <origin rpy="0 1.57075 0" xyz="0 0 -0.3"/>
-      <material name="white"/>
-    </visual>
-  </link>
-  <joint name="base_to_left_leg" type="fixed">
-    <parent link="base_link"/>
-    <child link="left_leg"/>
-    <origin xyz="0 0.22 0.25"/>
-  </joint>
-  <link name="left_base">
-    <visual>
-      <geometry>
-        <box size="0.4 0.1 0.1"/>
-      </geometry>
-      <material name="white"/>
-    </visual>
-  </link>
-  <joint name="left_base_joint" type="fixed">
-    <parent link="left_leg"/>
-    <child link="left_base"/>
-    <origin xyz="0 0 -0.6"/>
-  </joint>
-  <link name="left_front_wheel">
-    <visual>
-      <origin rpy="1.57075 0 0" xyz="0 0 0"/>
-      <geometry>
-        <cylinder length="0.1" radius="0.035"/>
-      </geometry>
-      <material name="black"/>
-    </visual>
-  </link>
-  <joint name="left_front_wheel_joint" type="fixed">
-    <parent link="left_base"/>
-    <child link="left_front_wheel"/>
-    <origin rpy="0 0 0" xyz="0.133333333333 0 -0.085"/>
-  </joint>
-  <link name="left_back_wheel">
-    <visual>
-      <origin rpy="1.57075 0 0" xyz="0 0 0"/>
-      <geometry>
-        <cylinder length="0.1" radius="0.035"/>
-      </geometry>
-      <material name="black"/>
-    </visual>
-  </link>
-  <joint name="left_back_wheel_joint" type="fixed">
-    <parent link="left_base"/>
-    <child link="left_back_wheel"/>
-    <origin rpy="0 0 0" xyz="-0.133333333333 0 -0.085"/>
-  </joint>
-  <joint name="gripper_extension" type="fixed">
-    <parent link="base_link"/>
-    <child link="gripper_pole"/>
-    <origin rpy="0 0 0" xyz="0.19 0 0.2"/>
-  </joint>
-  <link name="gripper_pole">
-    <visual>
-      <geometry>
-        <cylinder length="0.2" radius="0.01"/>
-      </geometry>
-      <origin rpy="0 1.57075 0 " xyz="0.1 0 0"/>
-    </visual>
-  </link>
-  <link name="head">
-    <visual>
-      <geometry>
-        <sphere radius="0.2"/>
-      </geometry>
-      <material name="white"/>
-    </visual>
-  </link>
-  <joint name="head_swivel" type="fixed">
-    <parent link="base_link"/>
-    <child link="head"/>
-    <origin xyz="0 0 0.3"/>
-  </joint>
-  <link name="box">
-    <visual>
-      <geometry>
-        <box size="0.08 0.08 0.08"/>
-      </geometry>
-      <material name="blue"/>
-    </visual>
-  </link>
-  <joint name="tobox" type="fixed">
-    <parent link="head"/>
-    <child link="box"/>
-    <origin xyz="0.1814 0 0.1414"/>
-  </joint>
-</robot>
+/home/ub2004/ros2_ws/build/urdf_tutorial/urdf/robot.xacro
